Commit message: Adds dynamic joint state publisher
Replaces the standard `joint_state_publisher` and static TF publishers for wheel drops.
Introduces a custom `dynamic_joint_state_publisher` node that subscribes to `/odom` and `/hazard_detection` topics to publish real-time joint states.
This enables dynamic visualization of:
- Wheel rotation based on odometry.
- Wheel drop status based on hazard detection.
- Bumper press status based on hazard detection.

Updates the bumper URDF to use a prismatic joint, allowing for its dynamic movement based on sensor data. This change provides a more accurate and responsive robot visualization.

File: create3_description/urdf/bumper.urdf.xacro (robot description, xacro)
@@ -17,8 +17,11 @@
   <xacro:property name="link_name" value="${name}"/>
   <xacro:property name="joint_name" value="${name}_joint"/>
-  <joint name="${joint_name}" type="fixed">
+  <joint name="${joint_name}" type="prismatic">
     <parent link="${parent_link}"/>
     <child link="${link_name}"/>
     <xacro:insert_block name="origin"/>
+    <axis xyz="1 0 0"/>
+    <limit lower="-0.003" upper="0" effort="0" velocity="0"/>
+    <dynamics damping="10" friction="0.1"/>
   </joint>
   <link name="${link_name}">
